File: docs/power_system/EPS/EPS_Scales_RevB/FPGA_WD.kicad_sch (KiCad schematic)
At the start: 40 parts, among them J6 Breakout, J7 Breakout, U3 TLV1704

Commit message: REV B. Schematic Finalized. Awaiting First Review
GPIO toggle pins added
Decoupling/filter caps added to power input.
Everything has been documented/added for clarification.
UV/OV resistors selected for Load Switches.
+5v Perif regulator tied to WDs and Clock. Slew rates calculated for 3 regulators and for 5v perif to setup phases prior to turning on.
Awaiting review.
Connections:
- net VCC_RF1 is gone; now on net +5V_ROUT3: JP5.1 (A)
Changed lines of the file:
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@@
 	(wire
 		(pts
-			(xy 30.48 45.72) (xy 30.48 46.99)
+			(xy 30.48 39.37) (xy 30.48 46.99)
 		)
 		(stroke
@@
 		)
 	)
-	(global_label "VCC_RF1"
-		(shape output)
-		(at 259.08 46.99 90)
+	(global_label "+5V_PerifOUT"
+		(shape input)
+		(at 240.03 52.07 0)
 		(fields_autoplaced yes)
 		(effects
@@
 		)
 		(property "Intersheetrefs" "${INTERSHEET_REFS}"
-			(at 259.08 35.8405 90)
+			(at 255.9572 52.07 0)
+			(effects
+				(font
+					(size 1.27 1.27)
+				)
+				(justify left)
+				(hide yes)
+			)
+		)
+	)
+	(global_label "+5V_PerifOUT"
+		(shape input)
+		(at 259.08 46.99 0)
+		(fields_autoplaced yes)
+		(effects
+			(font
+				(size 1.27 1.27)
+			)
+			(justify left)
+		)
+		(property "Intersheetrefs" "${INTERSHEET_REFS}"
+			(at 275.0072 46.99 0)
+			(effects
+				(font
+					(size 1.27 1.27)
+				)
+				(justify left)
+				(hide yes)
+			)
+		)
+	)
+	(global_label "+5V_PerifOUT"
+		(shape input)
+		(at 30.48 39.37 0)
+		(fields_autoplaced yes)
+		(effects
+			(font
+				(size 1.27 1.27)
+			)
+			(justify left)
+		)
+		(property "Intersheetrefs" "${INTERSHEET_REFS}"
+			(at 46.4072 39.37 0)
 			(effects
 				(font
@@
 		)
 	)
+	(global_label "+5V_PerifOUT"
+		(shape input)
+		(at 186.69 21.59 0)
+		(fields_autoplaced yes)
+		(effects
+			(font
+				(size 1.27 1.27)
+			)
+			(justify left)
+		)
+		(property "Intersheetrefs" "${INTERSHEET_REFS}"
+			(at 202.6172 21.59 0)
+			(effects
+				(font
+					(size 1.27 1.27)
+				)
+				(justify left)
+				(hide yes)
+			)
+		)
+	)
 	(symbol
 		(lib_id "Device:R_Small_US")
@@
 	(symbol
 		(lib_id "power:VBUS")
-		(at 30.48 45.72 0)
+		(at 30.48 39.37 0)
 		(unit 1)
 		(exclude_from_sim no)
@@
 		(dnp no)
 		(property "Reference" "#PWR029"
-			(at 30.48 49.53 0)
+			(at 30.48 43.18 0)
 			(effects
 				(font
@@
 		)
 		(property "Value" "+5V_ROUT3"
-			(at 29.21 40.894 0)
+			(at 29.21 34.544 0)
 			(effects
 				(font
@@
 				)
 				(justify left)
+				(hide yes)
 			)
 		)
 		(property "Footprint" ""
-			(at 30.48 45.72 0)
+			(at 30.48 39.37 0)
 			(effects
 				(font
@@
 		)
 		(property "Datasheet" ""
-			(at 30.48 45.72 0)
+			(at 30.48 39.37 0)
 			(effects
 				(font
@@
 		)
 		(property "Description" "Power symbol creates a global label with name \"VBUS\""
-			(at 30.48 45.72 0)
+			(at 30.48 39.37 0)
 			(effects
 				(font
@@
 				)
 				(justify left)
+				(hide yes)
 			)
 		)
@@
 				)
 				(justify left)
+				(hide yes)
 			)
 		)
