File: power_system/EPS/EPS_Voyager_RevA/EPS_Voyager/EPS_Voyager.kicad_pcb (KiCad board)
At the start: 4 copper layers, 75.2 x 28.2 mm, 52 parts, among them J1 Conn_01x02_Socket, J10 Conn_01x02_Socket, J11 Conn_01x02_Socket, J13 Conn_01x01_Socket, J14 Conn_01x02_Socket, J15 Conn_01x02_Socket, J16 Conn_01x04_Socket, J17 Conn_01x02_Socket, J18 Conn_01x02_Socket, J2 Input Power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

Commit message: Final Draft of EPS Voyager Complete
Basic board using 4 layers similar to what the final board will use. Uses 2.54mm headers for all configurable components. Awaiting review.
Parts:
- added TP23: TestPoint, TestPoint:TestPoint_Pad_1.0x1.0mm, F.Cu at (123.2, 41.0)
- moved R1 0.84 mm to (174.7, 52.1)
- moved R2 0.84 mm to (176.3, 52.1)
- moved U4 0.27 mm to (135.1, 44.0)
Routing:
- net +3.3V: track 0.00 -> 76.8 mm, vias 0 -> 1
- net Net-(J10-Pin_1): track 0.00 -> 71.5 mm, vias 0 -> 3
- net GND: track 0.00 -> 58.3 mm, vias 0 -> 20
- net Net-(U4-Vout): track 0.00 -> 42.9 mm, vias 0 -> 2
- net +V_Batt: track 0.00 -> 32.0 mm, vias 0 -> 1
- net Net-(J17-Pin_1): track 0.00 -> 24.2 mm
- net Net-(J3-Pin_2): track 0.00 -> 20.1 mm, vias 0 -> 2
- net Net-(J6-Pin_2): track 0.00 -> 18.9 mm, vias 0 -> 2
- net Net-(J8-Pin_2): track 0.00 -> 17.8 mm, vias 0 -> 1
- net Net-(J3-Pin_1): track 0.00 -> 17.5 mm, vias 0 -> 2
- net Net-(J4-Pin_1): track 0.00 -> 15.1 mm, vias 0 -> 1
- net +Vout: track 0.00 -> 13.7 mm, vias 0 -> 2
- net ~{LS_Toggle_GPIO}: track 0.00 -> 11.4 mm
- net SYNC_PHASE: track 0.00 -> 11.2 mm
- net OBC SDA: track 0.00 -> 10.2 mm, vias 0 -> 1
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Other:
- board size 75.2 x 28.2 mm -> 75.2 x 27.7 mm
- board text added: "EPS Voyager V1"
