File: power_system/EPS/EPS_Scales_RevC/EPS_Scales_RevC/EPS_Scales_RevC.kicad_sch (KiCad schematic)
At the start: 8 parts, among them J1 Input Power, J2 Conn_01x01_Socket, J3 Conn_01x01_Socket, J4 Conn_01x01_Socket, J5 Conn_01x01_Socket

Commit message: Rev C Schematic DONE
Components were finalized in meeting with Andrew Greenberg today, footprints have been assigned and specific component sizes and values have also been confirmed. Moving to layout for the first dev board of the SCALES EPS board.
Parts:
- C1, C2, C3: footprint Capacitor_SMD:C_1210_3225Metric -> Resistor_SMD:R_1210_3225Metric
Changed lines of the file:
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@@
 			)
 		)
-		(property "Footprint" "Capacitor_SMD:C_1210_3225Metric"
+		(property "Footprint" "Resistor_SMD:R_1210_3225Metric"
 			(at 168.6052 39.37 0)
 			(effects
@@
 			)
 		)
-		(property "Footprint" "Capacitor_SMD:C_1210_3225Metric"
+		(property "Footprint" "Resistor_SMD:R_1210_3225Metric"
 			(at 178.7652 39.37 0)
 			(effects
@@
 			)
 		)
-		(property "Footprint" "Capacitor_SMD:C_1210_3225Metric"
+		(property "Footprint" "Resistor_SMD:R_1210_3225Metric"
 			(at 173.6852 39.37 0)
 			(effects

Commit message: Rev C Layout #2 electric boogaloo
Yes
Parts:
- C1, C2, C3: value 10uF -> 10u; footprint Resistor_SMD:R_1210_3225Metric -> Capacitor_SMD:C_1210_3225Metric
Changed lines of the file:
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@@
 			)
 		)
-		(property "Value" "10uF"
+		(property "Value" "10u"
 			(at 165.608 28.448 0)
 			(effects
@@
 			)
 		)
-		(property "Footprint" "Resistor_SMD:R_1210_3225Metric"
+		(property "Footprint" "Capacitor_SMD:C_1210_3225Metric"
 			(at 168.6052 39.37 0)
 			(effects
@@
 			)
 		)
-		(property "Value" "10uF"
+		(property "Value" "10u"
 			(at 175.768 28.448 0)
 			(effects
@@
 			)
 		)
-		(property "Footprint" "Resistor_SMD:R_1210_3225Metric"
+		(property "Footprint" "Capacitor_SMD:C_1210_3225Metric"
 			(at 178.7652 39.37 0)
 			(effects
@@
 			)
 		)
-		(property "Value" "10uF"
+		(property "Value" "10u"
 			(at 170.688 28.448 0)
 			(effects
@@
 			)
 		)
-		(property "Footprint" "Resistor_SMD:R_1210_3225Metric"
+		(property "Footprint" "Capacitor_SMD:C_1210_3225Metric"
 			(at 173.6852 39.37 0)
 			(effects

Commit message: Minor changes to schematic
Changed lines of the file:
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@@
 		)
 	)
-	(text_box "Capacitors: 75v rated, 10uF ceramic, 3225 metric package\nDatasheeet in hyperlink"
+	(text_box "Capacitors for higher voltage lines: 75v rated, 10uF ceramic, 3225 metric package\nDatasheeet in hyperlink"
 		(exclude_from_sim no)
 		(at 135.255 49.53 0)
@@
 		)
 		(property "Value" "Input Power"
-			(at 186.69 26.162 0)
-			(effects
-				(font
+			(at 194.564 24.384 0)
+			(effects
+				(font
