File: power_system/EPS/EPS_Scales_RevC/EPS_Scales_RevC/EPS_Scales_RevC.kicad_pcb (KiCad board)
At the start: 4 copper layers, 111.8 x 64.7 mm, 249 parts, among them J1 Input Power, J10 DF11-16DP-2DSA, J11 DN-T1-GE3_VIS, J12 DF11-16DP-2DSA, J15 DN-T1-GE3_VIS, J16 Conn_01x04, J18 Conn_01x04, J2 Conn_01x01_Socket, J3 Conn_01x01_Socket, J4 Conn_01x01_Socket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

Commit message: Fixed Layout errors
Fixed Solder mask expansion errors
Added signature on board
Routing:
- net +3.3V_OBC: track 235.1 -> 239.1 mm
- net SYNC_PHASE3: track 83.0 -> 86.5 mm
- net SYNC_PHASE1: track 63.3 -> 66.8 mm
Other:
- board text added: "SCALES EPS Development Board By Luca Lanzillotta"
Changed lines of the file:
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@@
 			(pinfunction "GND")
 			(pintype "power_in")
-			(solder_mask_margin 0.102)
+			(solder_mask_margin 0.01)
 		)
 		(pad "1" smd rect
@@
 			(pinfunction "GND")
 			(pintype "power_in")
-			(solder_mask_margin 0.102)
+			(solder_mask_margin 0.01)
 		)
 		(pad "2" smd rect
@@
 			(pinfunction "OV")
 			(pintype "input")
-			(solder_mask_margin 0.102)
+			(solder_mask_margin 0.01)
 		)
 		(pad "3" smd rect
@@
 			(pinfunction "UV")
 			(pintype "input")
-			(solder_mask_margin 0.102)
+			(solder_mask_margin 0.01)
 		)
 		(pad "4" smd rect
@@
 			(pinfunction "Vin")
 			(pintype "power_in")
-			(solder_mask_margin 0.102)
+			(solder_mask_margin 0.01)
 		)
 		(pad "5" smd rect
@@
 			(pinfunction "GATE")
 			(pintype "output")
-			(solder_mask_margin 0.102)
+			(solder_mask_margin 0.01)
 		)
 		(pad "6" smd rect
@@
 			(pinfunction "Vout")
 			(pintype "passive")
-			(solder_mask_margin 0.102)
+			(solder_mask_margin 0.01)
 		)
 		(pad "7" smd rect
@@
 			(pinfunction "~{FAULT}")
 			(pintype "output+no_connect")
-			(solder_mask_margin 0.102)
+			(solder_mask_margin 0.01)
 		)
 		(pad "8" smd rect
@@
 			(pinfunction "~{SHDN}")
 			(pintype "passive")
-			(solder_mask_margin 0.102)
+			(solder_mask_margin 0.01)
 		)
 		(embedded_fonts no)
@@
 			(pinfunction "GND")
 			(pintype "power_in")
-			(solder_mask_margin 0.102)
+			(solder_mask_margin 0.01)
 		)
 		(pad "1" smd rect
@@
 			(pinfunction "GND")
 			(pintype "power_in")
-			(solder_mask_margin 0.102)
+			(solder_mask_margin 0.01)
 		)
 		(pad "2" smd rect
@@
 			(pinfunction "OV")
 			(pintype "input")
-			(solder_mask_margin 0.102)
+			(solder_mask_margin 0.01)
 		)
 		(pad "3" smd rect
@@
 			(pinfunction "UV")
 			(pintype "input")
-			(solder_mask_margin 0.102)
+			(solder_mask_margin 0.01)
 		)
 		(pad "4" smd rect
@@
 			(pinfunction "Vin")
 			(pintype "power_in")
-			(solder_mask_margin 0.102)
+			(solder_mask_margin 0.01)
 		)
 		(pad "5" smd rect
@@
 			(pinfunction "GATE")
 			(pintype "output")
-			(solder_mask_margin 0.102)
+			(solder_mask_margin 0.01)
 		)
 		(pad "6" smd rect
@@
 			(pinfunction "Vout")
 			(pintype "passive")
-			(solder_mask_margin 0.102)
+			(solder_mask_margin 0.01)
 		)
 		(pad "7" smd rect
@@
 			(pinfunction "~{FAULT}")
 			(pintype "output+no_connect")
-			(solder_mask_margin 0.102)
+			(solder_mask_margin 0.01)
 		)
 		(pad "8" smd rect
@@
 			(pinfunction "~{SHDN}")
 			(pintype "passive")
-			(solder_mask_margin 0.102)
+			(solder_mask_margin 0.01)
 		)
 		(embedded_fonts no)
@@
 			(pinfunction "GND")
 			(pintype "power_in")
-			(solder_mask_margin 0.102)
+			(solder_mask_margin 0.01)
 		)
 		(pad "1" smd rect
@@
 			(pinfunction "GND")
 			(pintype "power_in")
-			(solder_mask_margin 0.102)
+			(solder_mask_margin 0.01)
 		)
 		(pad "2" smd rect
@@
 			(pinfunction "OV")
 			(pintype "input")
-			(solder_mask_margin 0.102)
+			(solder_mask_margin 0.01)
 		)
 		(pad "3" smd rect
@@
 			(pinfunction "UV")
 			(pintype "input")
-			(solder_mask_margin 0.102)
+			(solder_mask_margin 0.01)
 		)
 		(pad "4" smd rect
@@
 			(pinfunction "Vin")
 			(pintype "power_in")
-			(solder_mask_margin 0.102)
+			(solder_mask_margin 0.01)
 		)
 		(pad "5" smd rect
@@
 			(pinfunction "GATE")
 			(pintype "output")
-			(solder_mask_margin 0.102)
+			(solder_mask_margin 0.01)
 		)
 		(pad "6" smd rect
@@
 			(pinfunction "Vout")
 			(pintype "passive")
-			(solder_mask_margin 0.102)
+			(solder_mask_margin 0.01)
 		)
 		(pad "7" smd rect
@@
 			(pinfunction "~{FAULT}")
 			(pintype "output+no_connect")
-			(solder_mask_margin 0.102)
+			(solder_mask_margin 0.01)
 		)
 		(pad "8" smd rect
@@
 			(pinfunction "~{SHDN}")
 			(pintype "passive")
-			(solder_mask_margin 0.102)
+			(solder_mask_margin 0.01)
 		)
 		(embedded_fonts no)
@@
 		(layer "Edge.Cuts")
 	)
+	(gr_text "SCALES EPS Development Board\nBy Luca Lanzillotta"
+		(at 196.775 69.5 90)
+		(layer "F.SilkS")
+		(effects
+			(font
+				(size 1.2 1.2)
+				(thickness 0.3)
+				(bold yes)
+			)
+			(justify left bottom)
+		)
+	)
 	(segment
 		(start 97.697802 65.2542)
@@
 	)
 	(segment
-		(start 161.2755 88.135)
-		(end 160.1925 88.135)
+		(start 168.6225 86.385)
+		(end 162.54 86.385)
 		(width 0.254)
 		(layer "F.Cu")
@@
 	)
 	(segment
-		(start 168.6225 86.385)
-		(end 163.0255 86.385)
+		(start 158.63 88.135)
+		(end 157.8425 87.3475)
 		(width 0.254)
 		(layer "F.Cu")
@@
 	)
 	(segment
-		(start 163.0255 86.385)
-		(end 161.2755 88.135)
+		(start 168.6425 85.3475)
+		(end 168.6225 85.3675)
 		(width 0.254)
 		(layer "F.Cu")
@@
 	)
 	(segment
-		(start 158.63 88.135)
-		(end 157.8425 87.3475)
+		(start 168.6225 85.3675)
+		(end 168.6225 86.385)
 		(width 0.254)
 		(layer "F.Cu")
@@
 	)
 	(segment
-		(start 168.6225 85.3675)
-		(end 168.6425 85.3475)
+		(start 162.092656 73.235)
+		(end 161.6925 73.635156)
 		(width 0.254)
 		(layer "F.Cu")
@@
 	)
 	(segment
-		(start 162.092656 73.235)
-		(end 161.6925 73.635156)
+		(start 162.54 86.385)
+		(end 160.79 88.135)
 		(width 0.254)
 		(layer "F.Cu")
@@
 	)
 	(segment
-		(start 168.6225 86.385)
-		(end 168.6225 85.3675)
+		(start 160.79 88.135)
+		(end 160.1925 88.135)
 		(width 0.254)
 		(layer "F.Cu")
@@
 	)
 	(segment
+		(start 168.0675 33.2925)
+		(end 168.0675 32.4325)
+		(width 0.508)
+		(layer "In2.Cu")
+		(net 42)
+	)
+	(segment
 		(start 159.1175 51.2175)
 		(end 159.9925 50.3425)
@@
 	)
 	(segment
+		(start 166.0675 33.2925)
+		(end 166.0675 32.4325)
+		(width 0.508)
+		(layer "In2.Cu")
+		(net 42)
+	)
+	(segment
 		(start 156.9925 51.2175)
 		(end 159.1175 51.2175)
@@
 	)
 	(segment
+		(start 166.15 32.35)
+		(end 168.15 32.35)
+		(width 0.508)
+		(layer "In2.Cu")
+		(net 42)
+	)
+	(segment
 		(start 137.2 48.625)
 		(end 148.125 48.625)
@@
 	)
 	(segment
+		(start 168.0675 32.4325)
+		(end 168.15 32.35)
+		(width 0.508)
+		(layer "In2.Cu")
+		(net 42)
+	)
+	(segment
+		(start 166.0675 32.4325)
+		(end 166.15 32.35)
+		(width 0.508)
+		(layer "In2.Cu")
+		(net 42)
+	)
+	(segment
 		(start 132 48.55)
 		(end 130.3 50.25)
@@
 	)
 	(segment
-		(start 155.003376 60.0705)
-		(end 151.578084 60.0705)
+		(start 126.9 58.775)
+		(end 127.075 58.95)
 		(width 0.254)
 		(layer "B.Cu")
@@
 	)
 	(segment
-		(start 148.282584 58.95)
-		(end 127.075 58.95)
+		(start 158.9455 57.1225)
+		(end 164.859658 57.1225)
 		(width 0.254)
 		(layer "B.Cu")
@@
 	)
 	(segment
-		(start 164.859658 57.1225)
-		(end 158.9455 57.1225)
+		(start 158.606916 57.8887)
+		(end 158.9455 57.550116)
 		(width 0.254)
 		(layer "B.Cu")
@@
 	)
 	(segment
-		(start 157.185176 57.8887)
+		(start 151.578084 60.0705)
 		(end 155.003376 60.0705)
 		(width 0.254)
@@
 	)
 	(segment
-		(start 158.606916 57.8887)
-		(end 157.185176 57.8887)
+		(start 127.075 58.95)
+		(end 150.457584 58.95)
 		(width 0.254)
 		(layer "B.Cu")
@@
 	)
 	(segment
-		(start 165.7425 57.8925)
-		(end 165.629658 57.8925)
+		(start 155.003376 60.0705)
+		(end 157.185176 57.8887)
 		(width 0.254)
 		(layer "B.Cu")
@@
 	)
 	(segment
-		(start 151.578084 60.0705)
-		(end 151.375084 59.8675)
+		(start 150.457584 58.95)
+		(end 151.578084 60.0705)
 		(width 0.254)
 		(layer "B.Cu")
@@
 	)
 	(segment
-		(start 158.9455 57.550116)
-		(end 158.606916 57.8887)
-		(width 0.254)
+		(start 123.95 61.725)
+		(end 123.95 66.15)
+		(width 0.15)
 		(layer "B.Cu")
 		(net 48)
 	)
 	(segment
-		(start 123.95 61.725)
-		(end 123.95 66.15)
-		(width 0.15)
+		(start 165.629658 57.8925)
+		(end 165.7425 57.8925)
+		(width 0.254)
 		(layer "B.Cu")
 		(net 48)
 	)
 	(segment
-		(start 158.9455 57.1225)
-		(end 158.9455 57.550116)
+		(start 164.859658 57.1225)
+		(end 165.629658 57.8925)
 		(width 0.254)
 		(layer "B.Cu")
@@
 	)
 	(segment
-		(start 127.075 58.95)
-		(end 126.9 58.775)
+		(start 157.185176 57.8887)
+		(end 158.606916 57.8887)
 		(width 0.254)
 		(layer "B.Cu")
@@
 	)
 	(segment
-		(start 165.629658 57.8925)
-		(end 164.859658 57.1225)
+		(start 158.9455 57.550116)
+		(end 158.9455 57.1225)
 		(width 0.254)
 		(layer "B.Cu")
@@
 	)
 	(segment
+		(start 151.278 57.997)
+		(end 152.1955 58.9145)
+		(width 0.254)
+		(layer "B.Cu")
+		(net 51)
+	)
+	(segment
 		(start 156.381516 57.282366)
 		(end 156.7201 56.943782)
@@
 		(width 0.254)
 		(layer "B.Cu")
+		(net 51)
+	)
+	(segment
+		(start 152.1955 58.9145)
+		(end 154.3705 58.9145)
+		(width 0.254)
+		(layer "B.Cu")
