File: imx8x_carrier_board/imx8x_carrier_v1/Backup_Power.kicad_sch (KiCad schematic)
At the start: 0 parts

Commit message: Updated Schematic
Working on Micro SD card connector.
Working on implementing power connector. Still uncertain about some things I still need to implement. WIP
Other:
- note added: "IMX8X Backup Power (VBatt)"
Changed lines of the file:
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@@
 	(generator_version "9.0")
 	(paper "A4")
+	(text "IMX8X Backup Power (VBatt)"
+		(exclude_from_sim no)
+		(at 36.195 15.875 0)
+		(effects
+			(font
+				(size 2.032 2.032)
+				(thickness 0.4064)
+				(bold yes)
+			)
+		)
+	)
+	(text_box "Backup power is a simple 3.3v coin cell that keeps the SOM RTC on at all times. We are including this because why not."
+		(exclude_from_sim no)
+		(at 13.97 19.05 0)
+		(size 53.975 8.255)
+		(margins 0.9525 0.9525 0.9525 0.9525)
+		(stroke
+			(width 0)
+			(type solid)
+		)
+		(fill
+			(type none)
+		)
+		(effects
+			(font
+				(size 1.27 1.27)
+				(thickness 0.254)
+				(bold yes)
+			)
+			(justify left top)
+		)
+	)
 )
