File: peripheral_board/peripheral_board_v1a/peripheral_board_v1a/peripheral_board_v1a.kicad_pcb (KiCad board)
At the start: 6 copper layers, 100.2 x 100.1 mm, 219 parts, among them CN1 Power Board Connector, CN2 DF11-16DP-2DSA(08), J1 Conn_01x03_Pin, J2 Conn_01x06, J3 Conn_02x06_Odd_Even, J4 Conn_01x06, J5 USB_C_Receptacle_USB2.0_16P, J6 RJ45_Pulse_JXD6-0001NL, J7 RJ45_Pulse_JXD6-0001NL, J8 RJ45_Pulse_JXD6-0001NL, J9 RJ45_Pulse_JXD6-0001NL, SW1 EVPAA602W, SW2 EVPAA602W, SW3 3_Pin_Dip_Switch_DSWB03LHGET_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, SW4 EVPAA602W, U1 RP2350A_C42411118, U2 AZ1117CH-3.3TRG1, U3 W25Q128JVSIQTR, U4 W5500, U5 SN74AHC1G125DBVR, U6 AZ1117CH-1.2TRG1, U7 KSZ8795CLXIC, Y1 ABM8-272-T3, Y2 25MHz, Y3 ABMM-25.000MHZ-B2-T

Commit message: PCB Update
Got all the parts on the board placed. Now just finishing the routing for each interconnection.
Trying to maintain a side to side/up to down but the board kinda follows it. For each plane  there is fill zones that will be for the chip that is on the top. Some of the traces are just being fed to where they need to go but the important EMI signals are being contained to their guidelines.
I will need to look at the lengths of the traces to make sure they are kept around the same length.

Will need to go over the board with some other eyes to make sure its ok.

I made sure the Wiznet traces are the same as SALAD.
Parts:
- removed the C45 at (-53.1, 103.3)
- removed the C46 at (-30.1, 104.1)
- removed the C47 at (-51.8, 104.5)
- removed the C48 at (-28.8, 102.7)
- removed D4, D5: LED, LED_SMD:LED_0603_1608Metric
- removed R47: 330, Resistor_SMD:R_0603_1608Metric
- removed the R48 at (-37.6, 93.4)
- TP10, TP11, TP13, TP15, TP17, TP22, TP23, TP25, TP27, TP29, TP30, TP32, TP33: moved to B.Cu
- moved TP35 269.3 mm to (166.9, 83.8), turned to 0 degrees
- moved C57 268.8 mm to (124.1, 67.4)
- moved C58 268.8 mm to (124.1, 61.0)
- moved J6 268.8 mm to (109.1, 64.2)
- moved R49 268.8 mm to (124.7, 58.3)
- moved R50 268.8 mm to (124.7, 59.8)
- moved R51 268.8 mm to (124.7, 68.6)
- moved R52 268.8 mm to (124.7, 70.1)
- moved TP36 268.6 mm to (166.9, 85.8), turned to 180 degrees
- moved C59 267.5 mm to (124.0, 86.1)
- moved C60 267.5 mm to (124.0, 79.7)
- moved J7 267.5 mm to (108.9, 82.9)
- moved R55 267.5 mm to (124.6, 87.3)
- moved R56 267.5 mm to (124.6, 88.9)
- moved R53 267.5 mm to (124.6, 77.0)
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- renumbered C68 to C22, C67 to C23, C23 to C24, C24 to C25, C22 to C26, C26 to C27, C27 to C28, C25 to C29, C28 to C30, C29 to C31, C30 to C32, C31 to C33, C32 to C34, C33 to C35, C35 to C36, C36 to C37, C37 to C38, C38 to C39, C41 to C40, C49 to C41, C50 to C42, C51 to C43, C55 to C44, C52 to C45, C53 to C46, C54 to C47, C34 to C48, C39 to C49, C40 to C50, C56 to C51, C42 to C52, C57 to C53, C43 to C54, C44 to C55, C58 to C56, C59 to C57, C60 to C58, C61 to C59, C62 to C60, C63 to C61, C64 to C62, C65 to C63, C66 to C64, FB5 to FB3, FB3 to FB4, FB6 to FB5, FB4 to FB6, R39 to R34, R40 to R35, R35 to R36, R36 to R37, R37 to R38, R38 to R39, R41 to R40, R42 to R41, R43 to R42, R44 to R43, R45 to R44, R46 to R45, R49 to R48, R50 to R49, R51 to R50, R52 to R51, R53 to R52, R54 to R53, R55 to R54, R56 to R55, R57 to R56, R58 to R57, R59 to R58, R60 to R59, R61 to R60, R62 to R61, R63 to R62, R64 to R63, R65 to R64, U7 to U6, U6 to U7
Connections:
- CN1 pad 1: VCC -> +3V3
- CN1 pad 3: VCC -> +3V3
- CN1 pad 5: VCC -> +3V3
- CN1 pad 7: VCC -> +3V3
- J6 pad 9: LED1_0 -> LED1_1
- J7 pad 9: LED2_0 -> LED2_1
- J8 pad 9: LED3_0 -> LED3_1
- J9 pad 9: LED4_0 -> LED4_1
- R50 pad 1: LED1_0 -> LED1_1
- R54 pad 1: LED2_0 -> LED2_1
- R58 pad 1: LED3_0 -> LED3_1
- R62 pad 1: LED4_0 -> LED4_1
- U1 pad 25: SWDIO -> SWD
Routing:
- net GPIO22: track 1.31 -> 56.6 mm
- net GPIO26_ADC0: track 1.20 -> 55.8 mm
- net GPIO27_ADC1: track 1.43 -> 55.3 mm
- net GPIO23: track 2.19 -> 56.0 mm
- net GPIO28_ADC2: track 1.15 -> 51.7 mm
- net GPIO24: track 3.02 -> 53.1 mm
- net I2C1_SCL: track 1.36 -> 51.4 mm
- net TX1-: track 0.00 -> 49.9 mm, vias 0 -> 2
- net GPIO29_ADC3: track 1.11 -> 50.7 mm
- net I2C1_SDA: track 1.53 -> 51.1 mm
- net TX1+: track 0.00 -> 48.9 mm, vias 0 -> 2
- net GPIO25: track 3.71 -> 52.3 mm
- net TX4+: track 0.00 -> 48.3 mm, vias 0 -> 2
- net TX4-: track 0.00 -> 46.6 mm, vias 0 -> 2
- net RX4+: track 0.00 -> 46.5 mm, vias 0 -> 2
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- added copper zone on In2.Cu, net +3V3
- added copper zone on In1.Cu, net CGND
- added copper zone on In1.Cu, net Chassis_GND
- added copper zone on B.Cu, net GND
- added copper zone on In1.Cu, net GND
- added copper zone on In1.Cu, net GNDA
Other:
- board text added: "Port 4"
- board text removed: "Wiznet Port"
