File: imx8x_carrier_board/imx8x_carrier_v2/imx8x_carrier_v2.kicad_pcb (KiCad board)
At the start: 6 copper layers, 100 x 100 mm, 246 parts, among them CN1 DF11-16DP-2DSA(08), J1 BTH-070-02-L-D-A, J3 Conn_01x05_Pin, J4 BTH-070-02-L-D-A, J5 Conn_02x07_Counter_Clockwise, J6 Conn_02x07_Counter_Clockwise, J7 Conn_01x02_Pin, Q1 IRLML6401, Q2 BSS138, SW1 SW_DIP_x01, SW2 KMR221GLFS, U1 DP83867IRRGZR, U10 MCP1824T-ADJE/OT, U11 BD2204GUL-E2, U2 74AUP1G08, U3 74LVC2G07, U4 FT2232HL, U5 LP38693MP-ADJ/NOPB, U6 CAT93C66VI-GT3, U7 TXS0101DCKR, U8 TXS0101DCKR, U9 TLV71310PDQNR, Y1 25MHz, Y2 12MHz

Commit message: imx8 board v2 ethernet
Wired the ethernet to the SOM connector. Checked to make sure there is length matching. Will need to look over it again once the board is complete.
Parts:
- C1, C10, C11, C12, C13, C14, C15, C16, C17, C18, C2, C21, C22, C54, C55, C56, C57, C58, C9, Q1, Q2, R1, R10, R11, R114, R115, R116, R117, R12, R13, R137, R138, R14, R15, R16, R17, R18, R19, R2, R20, R21, R22, R23, R24, R25, R3, R4, R5, R6, R7, R8, R9, U1, U10, U2, U3, U9, Y1: moved to B.Cu
- C19, C20, C23, C24, C25, C26, C27, C28, C29, C3, C30, C31, C32, C4, C5, C6, C7, C8: moved to F.Cu
- moved J7 89.9 mm to (71.2, 72.0)
- moved J3 86.6 mm to (70.9, 80.0)
- moved R138 40.6 mm to (158.3, 99.8)
- moved R137 38.6 mm to (157.3, 99.8)
- moved R115 36.5 mm to (156.3, 99.8)
- moved R116 34.4 mm to (155.2, 99.8)
- moved C57 34.2 mm to (155.1, 92.3)
- moved R117 33.6 mm to (154.8, 94.3), turned to 0 degrees
- moved U10 33.5 mm to (154.8, 96.8), turned to 0 degrees
- moved C58 31.0 mm to (153.5, 92.3)
- moved C56 29.7 mm to (152.8, 99.6), turned to 180 degrees
- moved C28 29.5 mm to (152.7, 95.8)
- moved C27 29.4 mm to (152.7, 98.8)
- moved R30 27.0 mm to (135.3, 113.4)
- moved C25 26.5 mm to (151.3, 95.8)
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Routing:
- net GND: track 0.00 -> 87.9 mm, vias 0 -> 40
- net X_POR_B_1V8: track 0.00 -> 81.6 mm, vias 0 -> 2
- net VCC_3V3_OUT: track 0.00 -> 73.4 mm, vias 0 -> 3
- net VCC_ENET_2V5: track 0.00 -> 66.7 mm, vias 0 -> 7
- net GNDPWR: track 0.00 -> 60.1 mm
- net VDD_ETH_1V0: track 0.00 -> 56.7 mm, vias 0 -> 7
- net X_ETH0_B_TX_N: track 0.00 -> 47.4 mm, vias 0 -> 2
- net X_ETH0_D_RXDV_N: track 0.00 -> 46.6 mm, vias 0 -> 2
- net X_ETH0_B_TX_P: track 0.00 -> 46.5 mm, vias 0 -> 2
- net X_ETH0_C_TXCLK_N: track 0.00 -> 45.1 mm, vias 0 -> 3
- net X_ETH0_C_TXCLK_P: track 0.00 -> 45.0 mm, vias 0 -> 3
- net X_ETH_GPIO0: track 0.00 -> 44.2 mm, vias 0 -> 4
- net X_ETH0_A_TX_P: track 0.00 -> 43.2 mm, vias 0 -> 1
- net X_ETH0_A_TX_N: track 0.00 -> 42.9 mm, vias 0 -> 1
- net X_ETH0_D_RXDV_P: track 0.00 -> 42.6 mm, vias 0 -> 2
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- added copper zone on B.Cu, net GND
- added copper zone on In1.Cu, net GND
