File: imx8x_carrier_board/imx8x_eps_v1/SOM.kicad_sch (KiCad schematic)
At the start: 41 parts, among them J1 BTH-070-02-L-D-A, J4 BTH-070-02-L-D-A

Commit message: Refining Schematic Connections.
Connections:
- no-connect marks 84 -> 85
Changed lines of the file:
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@@
+		)
+	)
+	(text_box "09 reserved for jetson watchdog"
+		(exclude_from_sim no)
+		(at 252.476 183.896 0)
+		(size 20.828 4.572)
+		(margins 0.9525 0.9525 0.9525 0.9525)
+		(stroke
+			(width 0)
+			(type solid)
+		)
+		(fill
+			(type none)
+		)
+		(effects
+			(font
+				(size 1.27 1.27)
+			)
+			(justify left top)
 		)
 	)
@@
 	)
 	(no_connect
+		(at 251.46 195.58)
+	)
+	(no_connect

Commit message: EPS+IMX
FIxed connector conflicts, redefined GPIO values and established a better flow for visuals.
Connections:
- net VCC_3V3 renamed +3.3V_OBC
- no-connect marks 85 -> 84
Other:
- moved on the sheet: C70
