File: imx8x_carrier_board/imx8x_carrier_v3/imx_microSD.kicad_sch (KiCad schematic)
At the start: 24 parts, among them SW1 SW_DIP_x01, U11 BD2204GUL-E2

Commit message: Replaced USB with Through Hole Variant. Added Images. Found replacement for LQFN to QFN
Small board revision
Other:
- company: (none) -> Bronco Space Lab
Changed lines of the file:
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@@
 	(generator_version "9.0")
 	(paper "A4")
+	(title_block
+		(company "Bronco Space Lab")
+	)
 	(rectangle
 		(start 13.335 13.97)
