File: imx8x_carrier_board/imx8x_carrier_v3/imx_power.kicad_sch (KiCad schematic)
At the start: 4 parts, among them CN1 DF11-16DP-2DSA(08)

Commit message: Replaced USB with Through Hole Variant. Added Images. Found replacement for LQFN to QFN
Small board revision
Other:
- company: (none) -> Bronco Space Lab
Changed lines of the file:
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@@
 	(generator_version "9.0")
 	(paper "A5")
+	(title_block
+		(company "Bronco Space Lab")
+	)
 	(rectangle
 		(start 14.351 39.624)
