File: imx8x_eps_leviathan_v2/.history/imx8x_eps_leviathan_v2.kicad_sch (KiCad schematic)
At the start: 0 parts

Commit message: Goodies
Updated USB to USB C. Added Diodes for USB. Improved Layout. Ready for some routing.
Other:
- title: Leviathan V1 -> Leviathan V2
Changed lines of the file:
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@@
 	(paper "A5")
 	(title_block
-		(title "Leviathan V1")
-		(date "2025-10-29")
-		(rev "V1")
+		(title "Leviathan V2")
+		(date "2026-04-21")
+		(rev "V2")
 		(company "Bronco Space Lab")
-		(comment 1 "By Luca Lanzillotta & John Pollack")
+		(comment 1 "By Luca Lanzillotta")
 	)
 	(rectangle
