File: imx8x_eps_leviathan_v2/.history/Pgood_Power.kicad_sch (KiCad schematic)
At the start: 10 parts, among them U29 TPS22917DBVR, U30 TLV62569PDDCR

Commit message: Goodies
Updated USB to USB C. Added Diodes for USB. Improved Layout. Ready for some routing.
Parts:
- renumbered C126 to C130, C127 to C131, C128 to C132, C129 to C133, R6 to R212, R20 to R213, U29 to U31, U30 to U32
Changed lines of the file:
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@@
 		(dnp no)
 		(fields_autoplaced yes)
-		(property "Reference" "#PWR046"
+		(property "Reference" "#PWR0205"
 			(at 73.152 50.8 0)
 			(hide yes)
@@
 			(project "imx8x_eps_leviathan_v2"
 				(path "/bd3af9f3-19df-4a2f-8b54-98c48cea082e/1b5b2e76-614d-4307-9232-e06f7c77302d/bd950bac-c734-4938-bbb2-10284e743c57"
-					(reference "#PWR046")
+					(reference "#PWR0205")
 					(unit 1)
 				)
@@
 		(dnp no)
 		(fields_autoplaced yes)
-		(property "Reference" "C128"
+		(property "Reference" "C132"
 			(at 118.11 39.3699 0)
 			(show_name no)
@@
 			(project "imx8x_eps_leviathan_v2"
 				(path "/bd3af9f3-19df-4a2f-8b54-98c48cea082e/1b5b2e76-614d-4307-9232-e06f7c77302d/bd950bac-c734-4938-bbb2-10284e743c57"
-					(reference "C128")
+					(reference "C132")
 					(unit 1)
 				)
@@
 		(dnp no)
 		(fields_autoplaced yes)
-		(property "Reference" "R20"
+		(property "Reference" "R213"
 			(at 177.546 44.4499 0)
 			(show_name no)
@@
 			(project "imx8x_eps_leviathan_v2"
 				(path "/bd3af9f3-19df-4a2f-8b54-98c48cea082e/1b5b2e76-614d-4307-9232-e06f7c77302d/bd950bac-c734-4938-bbb2-10284e743c57"
-					(reference "R20")
+					(reference "R213")
 					(unit 1)
 				)
@@
 		(in_pos_files yes)
 		(dnp no)
-		(property "Reference" "C126"
+		(property "Reference" "C130"
 			(at 34.798 35.56 0)
 			(show_name no)
@@
 			(project "imx8x_eps_leviathan_v2"
 				(path "/bd3af9f3-19df-4a2f-8b54-98c48cea082e/1b5b2e76-614d-4307-9232-e06f7c77302d/bd950bac-c734-4938-bbb2-10284e743c57"
-					(reference "C126")
+					(reference "C130")
 					(unit 1)
 				)
@@
 		(dnp no)
 		(fields_autoplaced yes)
-		(property "Reference" "U29"
+		(property "Reference" "U31"
 			(at 73.152 22.606 0)
 			(show_name no)
@@
 			(project "imx8x_eps_leviathan_v2"
 				(path "/bd3af9f3-19df-4a2f-8b54-98c48cea082e/1b5b2e76-614d-4307-9232-e06f7c77302d/bd950bac-c734-4938-bbb2-10284e743c57"
-					(reference "U29")
+					(reference "U31")
 					(unit 1)
 				)
@@
 		(dnp no)
 		(fields_autoplaced yes)
-		(property "Reference" "C129"
+		(property "Reference" "C133"
 			(at 168.148 36.3219 0)
 			(show_name no)
@@
 			(project "imx8x_eps_leviathan_v2"
 				(path "/bd3af9f3-19df-4a2f-8b54-98c48cea082e/1b5b2e76-614d-4307-9232-e06f7c77302d/bd950bac-c734-4938-bbb2-10284e743c57"
-					(reference "C129")
+					(reference "C133")
 					(unit 1)
 				)
@@
 		(in_pos_files yes)
 		(dnp no)
-		(property "Reference" "C127"
+		(property "Reference" "C131"
 			(at 43.688 35.56 0)
 			(show_name no)
@@
 			(project "imx8x_eps_leviathan_v2"
 				(path "/bd3af9f3-19df-4a2f-8b54-98c48cea082e/1b5b2e76-614d-4307-9232-e06f7c77302d/bd950bac-c734-4938-bbb2-10284e743c57"
-					(reference "C127")
+					(reference "C131")
 					(unit 1)
 				)
@@
 		(dnp no)
 		(fields_autoplaced yes)
-		(property "Reference" "#PWR0176"
+		(property "Reference" "#PWR0208"
 			(at 146.05 57.15 0)
 			(hide yes)
@@
 			(project "imx8x_eps_leviathan_v2"
 				(path "/bd3af9f3-19df-4a2f-8b54-98c48cea082e/1b5b2e76-614d-4307-9232-e06f7c77302d/bd950bac-c734-4938-bbb2-10284e743c57"
-					(reference "#PWR0176")
+					(reference "#PWR0208")
 					(unit 1)
 				)
@@
 		(in_pos_files yes)
 		(dnp no)
-		(property "Reference" "#PWR0172"
+		(property "Reference" "#PWR0206"
 			(at 85.09 34.29 0)
 			(hide yes)
@@
 			(project "imx8x_eps_leviathan_v2"
 				(path "/bd3af9f3-19df-4a2f-8b54-98c48cea082e/1b5b2e76-614d-4307-9232-e06f7c77302d/bd950bac-c734-4938-bbb2-10284e743c57"
-					(reference "#PWR0172")
+					(reference "#PWR0206")
 					(unit 1)
 				)
@@
 		(dnp no)
 		(fields_autoplaced yes)
-		(property "Reference" "R6"
+		(property "Reference" "R212"
 			(at 177.546 34.2899 0)
 			(show_name no)
@@
 			(project "imx8x_eps_leviathan_v2"
 				(path "/bd3af9f3-19df-4a2f-8b54-98c48cea082e/1b5b2e76-614d-4307-9232-e06f7c77302d/bd950bac-c734-4938-bbb2-10284e743c57"
-					(reference "R6")
+					(reference "R212")
 					(unit 1)
 				)
@@
 		(dnp no)
 		(fields_autoplaced yes)
-		(property "Reference" "U30"
+		(property "Reference" "U32"
 			(at 146.05 23.622 0)
 			(show_name no)
@@
 			(project "imx8x_eps_leviathan_v2"
 				(path "/bd3af9f3-19df-4a2f-8b54-98c48cea082e/1b5b2e76-614d-4307-9232-e06f7c77302d/bd950bac-c734-4938-bbb2-10284e743c57"
-					(reference "U30")
+					(reference "U32")
 					(unit 1)
 				)
@@
 		(in_pos_files yes)
 		(dnp no)
-		(property "Reference" "#PWR0171"
+		(property "Reference" "#PWR0204"
 			(at 33.02 34.29 0)
 			(hide yes)
@@
 			(project "imx8x_eps_leviathan_v2"
 				(path "/bd3af9f3-19df-4a2f-8b54-98c48cea082e/1b5b2e76-614d-4307-9232-e06f7c77302d/bd950bac-c734-4938-bbb2-10284e743c57"
-					(reference "#PWR0171")
+					(reference "#PWR0204")
 					(unit 1)
 				)
@@
 		(in_pos_files yes)
 		(dnp no)
-		(property "Reference" "#PWR0175"
+		(property "Reference" "#PWR0207"
 			(at 114.3 35.56 0)
 			(hide yes)
@@
 			(project "imx8x_eps_leviathan_v2"
 				(path "/bd3af9f3-19df-4a2f-8b54-98c48cea082e/1b5b2e76-614d-4307-9232-e06f7c77302d/bd950bac-c734-4938-bbb2-10284e743c57"
-					(reference "#PWR0175")
+					(reference "#PWR0207")
 					(unit 1)
 				)
@@
 		(in_pos_files yes)
 		(dnp no)
-		(property "Reference" "#PWR0177"
+		(property "Reference" "#PWR0209"
 			(at 175.26 35.56 0)
 			(hide yes)
@@
 			(project "imx8x_eps_leviathan_v2"
 				(path "/bd3af9f3-19df-4a2f-8b54-98c48cea082e/1b5b2e76-614d-4307-9232-e06f7c77302d/bd950bac-c734-4938-bbb2-10284e743c57"
-					(reference "#PWR0177")
-					(unit 1)
-				)
+					(reference "#PWR0209")
+					(unit 1)
+				)

Commit message: Fixed Duplicates. Updated Gerber and BOM
Parts:
- C130: value 1uF -> 1u
- C131: value 47uF -> 47u
- C132: value 4.7uF -> 4.7u
- C133: value 10uF -> 10u
- L6: value 2.2uH -> 2.2u
Changed lines of the file:
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@@
 		(fields_autoplaced yes)
 		(property "Reference" "L6"
-			(at 158.75 26.416 90)
-			(show_name no)
-			(do_not_autoplace no)
-			(effects
-				(font
-					(size 1.27 1.27)
-				)
-			)
-		)
-		(property "Value" "2.2uH"
-			(at 158.75 28.956 90)
+			(at 158.75 26.67 90)
+			(show_name no)
+			(do_not_autoplace no)
+			(effects
+				(font
+					(size 1.27 1.27)
+				)
+			)
+		)
+		(property "Value" "2.2u"
+			(at 158.75 29.21 90)
 			(show_name no)
 			(do_not_autoplace no)
@@
 			)
 		)
-		(property "Value" "4.7uF"
+		(property "Value" "4.7u"
 			(at 118.11 41.9099 0)
 			(show_name no)
@@
 			)
 		)
-		(property "Value" "1uF"
+		(property "Value" "1u"
 			(at 34.798 39.624 0)
 			(show_name no)
@@
 		(fields_autoplaced yes)
 		(property "Reference" "C133"
-			(at 168.148 36.3219 0)
-			(show_name no)
-			(do_not_autoplace no)
-			(effects
-				(font
-					(size 1.27 1.27)
-				)
-				(justify left)
-			)
-		)
-		(property "Value" "10uF"
-			(at 168.148 38.8619 0)
+			(at 167.64 36.3219 0)
+			(show_name no)
+			(do_not_autoplace no)
+			(effects
+				(font
+					(size 1.27 1.27)
+				)
+				(justify left)
+			)
+		)
+		(property "Value" "10u"
+			(at 167.64 38.8619 0)
 			(show_name no)
 			(do_not_autoplace no)
@@
 			)
 		)
-		(property "Value" "47uF"
+		(property "Value" "47u"
 			(at 43.688 39.624 0)
 			(show_name no)
