File: imx8x_eps_leviathan_v2/.history/WD_Jetson.kicad_sch (KiCad schematic)
At the start: 32 parts, among them U17 TLV1704

Commit message: Goodies
Updated USB to USB C. Added Diodes for USB. Improved Layout. Ready for some routing.
Parts:
- renumbered C50 to C49, C51 to C50, C52 to C51, C53 to C52, C54 to C53, C55 to C54, C56 to C55, C57 to C56, D7 to D4, D8 to D5, D9 to D6, R66 to R63, R67 to R64, R68 to R65, R69 to R66, R70 to R67, R71 to R68, R72 to R69, R73 to R70, R74 to R71, R75 to R72, R76 to R73, R77 to R74, R78 to R75, R79 to R76, R80 to R77, R81 to R78, R82 to R79, R83 to R80, TP42 to TP20
Connections:
- net ~{WD_EN_JETSON}: no longer JP2.2 (B)
- net at JP2.1 (A): no longer U17.13
Other:
- title: Leviathan V1 -> Leviathan V2

Commit message: Continued Layout
Connections:
- net ~{WD_EN_JETSON}: now also JP2.2 (B)
- net at JP2.1 (A): now also U17.13
Other:
- moved on the sheet: JP2
Changed lines of the file:
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@@
-	(wire
-		(pts
-			(xy 266.7 120.65) (xy 266.7 123.19)
-		)
-		(stroke
-			(width 0)
-			(type default)
-		)
-	)
 	(wire
 		(pts
@@
 	(symbol
 		(lib_id "Jumper:SolderJumper_2_Open")
-		(at 266.7 116.84 270)
+		(at 266.7 118.11 270)
 		(unit 1)
 		(body_style 1)
@@
 		(dnp no)
 		(property "Reference" "JP2"
-			(at 263.906 117.094 0)
+			(at 263.906 118.364 0)
 			(show_name no)
 			(do_not_autoplace no)
@@
 		)
 		(property "Value" "SolderJumper_2_Open"
-			(at 280.67 116.84 90)
+			(at 280.67 118.11 90)
 			(hide yes)
 			(show_name no)
@@
 		)
 		(property "Footprint" "Jumper:SolderJumper-2_P1.3mm_Open_RoundedPad1.0x1.5mm"
-			(at 266.7 116.84 0)
+			(at 266.7 118.11 0)
 			(hide yes)
 			(show_name no)
@@
 		)
 		(property "Datasheet" ""
-			(at 266.7 116.84 0)
+			(at 266.7 118.11 0)
 			(hide yes)
 			(show_name no)
@@
 		)
 		(property "Description" "Solder Jumper, 2-pole, open"
-			(at 266.7 116.84 0)
-			(hide yes)
-			(show_name no)
+			(at 266.7 118.11 0)
+			(hide yes)
+			(show_name no)

Commit message: Fixed an ERC error, and updated reference designators so there are no more conflicts
Parts:
- C49, C50, C51: value 100uF -> 100u
Changed lines of the file:
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@@
 			)
 		)
-		(property "Value" "100uF"
+		(property "Value" "100u"
 			(at 43.18 58.4199 90)
 			(show_name no)
@@
 			)
 		)
-		(property "Value" "100uF"
+		(property "Value" "100u"
 			(at 24.13 58.4199 90)
 			(show_name no)
@@
 			)
 		)
-		(property "Value" "100uF"
+		(property "Value" "100u"
 			(at 33.02 58.4199 90)
 			(show_name no)
